File: project/pcb/redesign/buck.kicad_sch (KiCad schematic)
At the start: 0 parts

Commit message: feat: Buck PCB Rev B prototype package for JLCPCB
Rev B of project/pcb/redesign, prepared for a JLCPCB top-side SMT quote
and still pending bring-up. Rev A is preserved in history/revA_quote_20261027.

- Lands taken from manufacturer drawings (Murata 6000B, Same Sky TB002,
  Wurth WR-BHD, Panasonic SVPF/SVF, TA-I RLP, TI PW/DBV/DBZ/D/DBV5, Diodes
  SOD323); Q1 hole 1.4 mm per IPC-2222; U5 courtyard added.
- Power-domain interface: SN74LV4T125 buffer for PWM/RUN/RESET from +5V,
  TMUX1511 on the ADC path, TPS3808G33 supervisor, LM4040 2.5 V reference
  with BAT54WS clamps, fault latch set while the interface is disabled.
- Re-laid board: compact switching cell, no vias on HO/GATE/BOOT/SW,
  Kelvin sensing from RS1 inner edges, GND pours on both layers.
- L432KC firmware: Rev B ADC scale (6.4844 mV/count), VOUT-collapse fault,
  host test.
- Fabrication package production/jlcpcb-revB-2026-10-27: DRC 0 errors,
  0 unconnected, 0 parity; ERC 0 errors.

Not ready to order: L1/L2 have no JLC/LCSC stock, the LM4040 X-variant and
R10 supply need decisions, the JLC viewer rotation check and ARM build are
pending. BUCK_BOARD_REVIEWED stays 0. See revB_release_report.md.

Co-Authored-By: Claude Opus 5.5 <noreply@anthropic.com>
Other:
- added sheet Power-domain interface (buck_5.kicad_sch)
- title: Buck 12V / 6V - REVIEW ONLY -> Buck 12V / 6V - REV B PROTOTYPE
Changed lines of the file:
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@@
   (paper "A4")
   (title_block
-    (title "Buck 12V / 6V - REVIEW ONLY")
-    (rev "A")
+    (title "Buck 12V / 6V - REV B PROTOTYPE")
+    (rev "B")
     (company "UNAL Manizales")
   )
@@
     )
   )
+  (sheet (at 30 155) (size 130 18) (exclude_from_sim no) (in_bom yes) (on_board yes) (dnp no) (stroke (width 0.1524) (type solid)) (fill (color 0 0 0 0)) (property "Sheetname" "Power-domain interface" (at 30 154 0) (show_name no) (do_not_autoplace no) (effects (font (size 1.27 1.27)))) (property "Sheetfile" "buck_5.kicad_sch" (at 30 175 0) (show_name no) (do_not_autoplace no) (effects (font (size 1.27 1.27)))) (instances (project "buck" (path "/94b2b377-c0d1-5fce-91fa-ae8f86f36484" (page "6")))))
   (sheet_instances
     (path "/"
