File: project/pcb/redesign/buck_3.kicad_sch (KiCad schematic)
At the start: 17 parts, among them Q2 MMBT3904, U4 SN74HCT00DR, U5 LM393BIDR, U6 INA180A1IDBVR

Commit message: feat: Buck PCB Rev B prototype package for JLCPCB
Rev B of project/pcb/redesign, prepared for a JLCPCB top-side SMT quote
and still pending bring-up. Rev A is preserved in history/revA_quote_20261027.

- Lands taken from manufacturer drawings (Murata 6000B, Same Sky TB002,
  Wurth WR-BHD, Panasonic SVPF/SVF, TA-I RLP, TI PW/DBV/DBZ/D/DBV5, Diodes
  SOD323); Q1 hole 1.4 mm per IPC-2222; U5 courtyard added.
- Power-domain interface: SN74LV4T125 buffer for PWM/RUN/RESET from +5V,
  TMUX1511 on the ADC path, TPS3808G33 supervisor, LM4040 2.5 V reference
  with BAT54WS clamps, fault latch set while the interface is disabled.
- Re-laid board: compact switching cell, no vias on HO/GATE/BOOT/SW,
  Kelvin sensing from RS1 inner edges, GND pours on both layers.
- L432KC firmware: Rev B ADC scale (6.4844 mV/count), VOUT-collapse fault,
  host test.
- Fabrication package production/jlcpcb-revB-2026-10-27: DRC 0 errors,
  0 unconnected, 0 parity; ERC 0 errors.

Not ready to order: L1/L2 have no JLC/LCSC stock, the LM4040 X-variant and
R10 supply need decisions, the JLC viewer rotation check and ARM build are
pending. BUCK_BOARD_REVIEWED stays 0. See revB_release_report.md.

Co-Authored-By: Claude Opus 5.5 <noreply@anthropic.com>
Parts:
- U4: footprint Buck_SMD:D14 -> Buck_RevB:TI_D0014A_SOIC-14; Migration_Status FOOTPRINT_ONLY / PROVISIONAL - REVIEW REQUIRED -> REV B - LAND CORRECTED TO MANUFACTURER DRAWING
- U5: footprint Buck_SMD:D0008A-MFG -> Buck_RevB:TI_D0008A_SOIC-8; Migration_Status FOOTPRINT_ONLY / PROVISIONAL - REVIEW REQUIRED -> REV B - LAND CORRECTED TO MANUFACTURER DRAWING
- U6: footprint Buck_SMD:DBV0005A_N -> Buck_RevB:TI_DBV0005A_SOT-23-5; Migration_Status FOOTPRINT_ONLY / PROVISIONAL - REVIEW REQUIRED -> REV B - LAND CORRECTED TO MANUFACTURER DRAWING
Connections:
- net RESET: no longer U4.1 (1A)
- net RUN: no longer U4.4 (2A)
- new net RESET_5V: U4.1 (1A)
- new net RUN_5V: U4.4 (2A)
Other:
- title: Independent protection - REV A / HOLD FABRICATION -> Independent protection - REV B PROTOTYPE
Changed lines of the file:
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@@
   (paper "A3")
   (title_block
-    (title "Independent protection - REV A / HOLD FABRICATION")
-    (rev "A")
+    (title "Independent protection - REV B PROTOTYPE")
+    (rev "B")
     (company "UNAL Manizales - Sistemas Dinamicos y Control")
   )
@@
     )
   )
-  (global_label "RESET"
+  (global_label "RESET_5V"
     (shape passive)
     (at 33.02 29.21 180)
@@
     )
   )
-  (global_label "RUN"
+  (global_label "RUN_5V"
     (shape passive)
     (at 33.02 36.83 180)
@@
       )
     )
-    (property "Footprint" "Buck_SMD:DBV0005A_N"
+    (property "Footprint" "Buck_RevB:TI_DBV0005A_SOT-23-5"
       (at 50.8 165.1 0)
       (hide yes)
@@
       )
     )
-    (property "Migration_Status" "FOOTPRINT_ONLY / PROVISIONAL - REVIEW REQUIRED"
+    (property "Migration_Status" "REV B - LAND CORRECTED TO MANUFACTURER DRAWING"
       (at 50.8 165.1 0)
       (effects
@@
       )
     )
-    (property "Footprint" "Buck_SMD:D14"
+    (property "Footprint" "Buck_RevB:TI_D0014A_SOIC-14"
       (at 50.8 35.56 0)
       (hide yes)
@@
       )
     )
-    (property "Migration_Status" "FOOTPRINT_ONLY / PROVISIONAL - REVIEW REQUIRED"
+    (property "Migration_Status" "REV B - LAND CORRECTED TO MANUFACTURER DRAWING"
       (at 50.8 35.56 0)
       (effects
@@
       )
     )
-    (property "Footprint" "Buck_SMD:D0008A-MFG"
+    (property "Footprint" "Buck_RevB:TI_D0008A_SOIC-8"
       (at 149.86 78.74 0)
       (hide yes)
@@
       )
     )
-    (property "Migration_Status" "FOOTPRINT_ONLY / PROVISIONAL - REVIEW REQUIRED"
+    (property "Migration_Status" "REV B - LAND CORRECTED TO MANUFACTURER DRAWING"
       (at 149.86 78.74 0)
       (effects

Commit message: fix: make Buck Rev B orderable as a lab prototype
Order decisions after an external second opinion:
- Move the L1-L2-RS1-output chain 2 mm right: Q1 tab (VIN) to L1 SW clip
  clearance 1.28 -> 3.29 mm at maximum package dimensions; board rerouted,
  DRC 0 errors / 0 unconnected / 0 parity.
- L1/L2 (60B334C, no JLC/LCSC stock) leave the JLC BOM/CPL and are
  hand-soldered: 31 BOM lines, 62 placements, all with JLC stock.
- R10 -> UNI-ROYAL 0603WAF3092T5E (C23022), same 30.9k 1% 0603.
- Accept LM4040AIM3X-2.5/NOPB (same device per TI SNOS633N s.11).
- Document lab-only use: regulated 12 V, resistive load, supervised tests.

Co-Authored-By: Claude Opus 5.5 <noreply@anthropic.com>
Parts:
- R10: Commercial_URL https://jlcpcb.com/partdetail/VishayIntertech-CRCW060330K9F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 -> https://jlcpcb.com/partdetail/C23022; LCSC C844354 -> C23022; MPN CRCW060330K9FKEA -> 0603WAF3092T5E; Manufacturer Vishay -> UNI-ROYAL; Substitution_Note (none) -> Rev B order: CRCW060330K9FKEA (C844354) had 5 in JLC stock;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
Changed lines of the file:
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@@
     (pin "2"
     )
+    (property "Substitution_Note" "Rev B order: CRCW060330K9FKEA (C844354) had 5 in JLC stock; same 30.9k 1% 0603, +-100 ppm" (at 248.92 121.92 0) (hide yes) (effects (font (size 1.27 1.27))))
     (instances
       (project "buck"
@@
       )
     )
-    (property "MPN" "CRCW060330K9FKEA"
+    (property "MPN" "0603WAF3092T5E"
       (at 248.92 121.92 0)
       (effects
@@
       )
     )
-    (property "LCSC" "C844354"
+    (property "LCSC" "C23022"
       (at 248.92 121.92 0)
       (effects
@@
       )
     )
-    (property "Manufacturer" "Vishay"
+    (property "Manufacturer" "UNI-ROYAL"
       (at 248.92 121.92 0)
       (effects
@@
       )
     )
-    (property "Commercial_URL" "https://jlcpcb.com/partdetail/VishayIntertech-CRCW060330K9FKEA/C844354"
+    (property "Commercial_URL" "https://jlcpcb.com/partdetail/C23022"
       (at 248.92 121.92 0)
       (effects
