File: project/pcb/redesign/buck_1.kicad_sch (KiCad schematic)
At the start: 12 parts, among them J1 12V FUSED INPUT, J2 LOAD + / -, Q1 IRFZ44N TO-220

Commit message: feat: Buck PCB Rev B prototype package for JLCPCB
Rev B of project/pcb/redesign, prepared for a JLCPCB top-side SMT quote
and still pending bring-up. Rev A is preserved in history/revA_quote_20261027.

- Lands taken from manufacturer drawings (Murata 6000B, Same Sky TB002,
  Wurth WR-BHD, Panasonic SVPF/SVF, TA-I RLP, TI PW/DBV/DBZ/D/DBV5, Diodes
  SOD323); Q1 hole 1.4 mm per IPC-2222; U5 courtyard added.
- Power-domain interface: SN74LV4T125 buffer for PWM/RUN/RESET from +5V,
  TMUX1511 on the ADC path, TPS3808G33 supervisor, LM4040 2.5 V reference
  with BAT54WS clamps, fault latch set while the interface is disabled.
- Re-laid board: compact switching cell, no vias on HO/GATE/BOOT/SW,
  Kelvin sensing from RS1 inner edges, GND pours on both layers.
- L432KC firmware: Rev B ADC scale (6.4844 mV/count), VOUT-collapse fault,
  host test.
- Fabrication package production/jlcpcb-revB-2026-10-27: DRC 0 errors,
  0 unconnected, 0 parity; ERC 0 errors.

Not ready to order: L1/L2 have no JLC/LCSC stock, the LM4040 X-variant and
R10 supply need decisions, the JLC viewer rotation check and ARM build are
pending. BUCK_BOARD_REVIEWED stays 0. See revB_release_report.md.

Co-Authored-By: Claude Opus 5.5 <noreply@anthropic.com>
Parts:
- C1, C2: footprint Buck_SMD:PCAP_SVP_E7_PAN -> Buck_RevB:CP_Panasonic_SVPF_E7_Land; Migration_Status FOOTPRINT_ONLY / PROVISIONAL - REVIEW REQUIRED -> REV B - LAND CORRECTED TO MANUFACTURER DRAWING
- C4, C5: value 10uF 35V low ESR -> 10uF 50V 50SVF10M; footprint Buck_SMD:CAP_SVF_C6_PAN -> Buck_RevB:CP_Panasonic_SVF_C6_Land; Migration_Status FOOTPRINT_ONLY / PROVISIONAL - REVIEW REQUIRED -> REV B - LAND CORRECTED TO MANUFACTURER DRAWING
- J1: value 12V FUSED INPUT -> 12V IN TB002-500-02BE; footprint TerminalBlock_Phoenix:TerminalBlock_Phoenix_MKDS-1,5-2_1x02_P5.00mm_Horizontal -> Buck_RevB:TerminalBlock_SameSky_TB002-500-02_1x02_P5.00mm; Assembly (none) -> MANUAL_THT; Electrical_Approval PENDING - NOT APPROVED -> PENDING - PROTOTYPE BRING-UP; NOT ELECTRICALLY VALIDATED; LCSC (none) -> C2757858; MPN (none) -> TB002-500-02BE; Manufacturer (none) -> Same Sky; Migration_Status PENDING / ORIGINAL RETAINED -> REV B - PART FIXED BY RELEASE PLAN
- J2: value LOAD + / - -> LOAD TB002-500-02BE; footprint TerminalBlock_Phoenix:TerminalBlock_Phoenix_MKDS-1,5-2_1x02_P5.00mm_Horizontal -> Buck_RevB:TerminalBlock_SameSky_TB002-500-02_1x02_P5.00mm; Assembly (none) -> MANUAL_THT; Electrical_Approval PENDING - NOT APPROVED -> PENDING - PROTOTYPE BRING-UP; NOT ELECTRICALLY VALIDATED; LCSC (none) -> C2757858; MPN (none) -> TB002-500-02BE; Manufacturer (none) -> Same Sky; Migration_Status PENDING / ORIGINAL RETAINED -> REV B - PART FIXED BY RELEASE PLAN
- L1, L2: value 330uH >=3A Isat VERIFY -> 330uH 60B334C; footprint Buck:Inductor_25mm_P10mm_VERIFY -> Buck_RevB:L_Murata_6000B_27.0x23.5mm; Assembly (none) -> JLC_SMT_TOP_SUPPLY_BLOCKED; Electrical_Approval PENDING - NOT APPROVED -> PENDING - PROTOTYPE BRING-UP; NOT ELECTRICALLY VALIDATED; LCSC (none) -> C6823957; MPN (none) -> 60B334C; Manufacturer (none) -> Murata Power Solutions; Migration_Status PENDING / ORIGINAL RETAINED -> REV B - PART FIXED BY RELEASE PLAN
- Q1: value IRFZ44N TO-220 -> IRFZ44NPBF; footprint Package_TO_SOT_THT:TO-220-3_Vertical -> Buck_RevB:TO-220-3_Vertical_Drill1.4; Assembly (none) -> MANUAL_THT; Electrical_Approval PENDING - NOT APPROVED -> PENDING - PROTOTYPE BRING-UP; NOT ELECTRICALLY VALIDATED; LCSC (none) -> C2586; MPN (none) -> IRFZ44NPBF; Manufacturer (none) -> Infineon; Migration_Status PENDING / ORIGINAL RETAINED -> REV B - PART FIXED BY RELEASE PLAN
- RS1: value 0.050R 1% 1W -> 0.050R 1% 2W RLP25FEER050; footprint Resistor_SMD:R_2512_6332Metric -> Buck_RevB:R_TAI_RLP25_2512_Kelvin; Migration_Status FOOTPRINT_ONLY / PROVISIONAL - REVIEW REQUIRED -> REV B - LAND CORRECTED TO MANUFACTURER DRAWING
Other:
- title: Power stage - REV A / HOLD FABRICATION -> Power stage - REV B PROTOTYPE
Changed lines of the file:
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@@
   (paper "A3")
   (title_block
-    (title "Power stage - REV A / HOLD FABRICATION")
-    (rev "A")
+    (title "Power stage - REV B PROTOTYPE")
+    (rev "B")
     (company "UNAL Manizales - Sistemas Dinamicos y Control")
   )
@@
       )
     )
-    (property "Value" "10uF 35V low ESR"
+    (property "Value" "10uF 50V 50SVF10M"
       (at 248.92 128.46 0)
       (show_name no)
@@
       )
     )
-    (property "Footprint" "Buck_SMD:CAP_SVF_C6_PAN"
+    (property "Footprint" "Buck_RevB:CP_Panasonic_SVF_C6_Land"
       (at 248.92 121.92 0)
       (hide yes)
@@
       )
     )
-    (property "Migration_Status" "FOOTPRINT_ONLY / PROVISIONAL - REVIEW REQUIRED"
+    (property "Migration_Status" "REV B - LAND CORRECTED TO MANUFACTURER DRAWING"
       (at 248.92 121.92 0)
       (effects
@@
       )
     )
-    (property "Value" "0.050R 1% 1W"
+    (property "Value" "0.050R 1% 2W RLP25FEER050"
       (at 149.86 85.28 0)
       (show_name no)
@@
       )
     )
-    (property "Footprint" "Resistor_SMD:R_2512_6332Metric"
+    (property "Footprint" "Buck_RevB:R_TAI_RLP25_2512_Kelvin"
       (at 149.86 78.74 0)
       (hide yes)
@@
       )
     )
-    (property "Migration_Status" "FOOTPRINT_ONLY / PROVISIONAL - REVIEW REQUIRED"
+    (property "Migration_Status" "REV B - LAND CORRECTED TO MANUFACTURER DRAWING"
       (at 149.86 78.74 0)
       (effects
@@
       )
     )
-    (property "Value" "12V FUSED INPUT"
+    (property "Value" "12V IN TB002-500-02BE"
       (at 50.8 42.1 0)
       (show_name no)
@@
       )
     )
-    (property "Footprint" "TerminalBlock_Phoenix:TerminalBlock_Phoenix_MKDS-1,5-2_1x02_P5.00mm_Horizontal"
+    (property "Footprint" "Buck_RevB:TerminalBlock_SameSky_TB002-500-02_1x02_P5.00mm"
       (at 50.8 35.56 0)
       (hide yes)
@@
       )
     )
-    (property "Datasheet" ""
+    (property "Datasheet" "https://www.sameskydevices.com/product/resource/tb002-500.pdf"
       (at 50.8 35.56 0)
       (show_name no)
@@
     (pin "1"
     )
+    (property "MPN" "TB002-500-02BE" (at 50.8 35.56 0) (hide yes) (effects (font (size 1.27 1.27)))) (property "Manufacturer" "Same Sky" (at 50.8 35.56 0) (hide yes) (effects (font (size 1.27 1.27)))) (property "LCSC" "C2757858" (at 50.8 35.56 0) (hide yes) (effects (font (size 1.27 1.27)))) (property "Assembly" "MANUAL_THT" (at 50.8 35.56 0) (hide yes) (effects (font (size 1.27 1.27))))
     (instances
       (project "buck"
@@
       )
     )
-    (property "Migration_Status" "PENDING / ORIGINAL RETAINED"
+    (property "Migration_Status" "REV B - PART FIXED BY RELEASE PLAN"
       (at 50.8 35.56 0)
       (effects
@@
       )
     )
-    (property "Electrical_Approval" "PENDING - NOT APPROVED"
+    (property "Electrical_Approval" "PENDING - PROTOTYPE BRING-UP; NOT ELECTRICALLY VALIDATED"
       (at 50.8 35.56 0)
       (effects
@@
       )
     )
-    (property "Value" "330uH >=3A Isat VERIFY"
+    (property "Value" "330uH 60B334C"
       (at 347.98 42.1 0)
       (show_name no)
@@
       )
     )
-    (property "Footprint" "Buck:Inductor_25mm_P10mm_VERIFY"
+    (property "Footprint" "Buck_RevB:L_Murata_6000B_27.0x23.5mm"
       (at 347.98 35.56 0)
       (hide yes)
@@
       )
     )
-    (property "Datasheet" ""
+    (property "Datasheet" "https://www.murata.com/products/power/power-magnetics (KMP_6000B_B01)"
       (at 347.98 35.56 0)
       (show_name no)
@@
     (pin "2"
     )
+    (property "MPN" "60B334C" (at 347.98 35.56 0) (hide yes) (effects (font (size 1.27 1.27)))) (property "Manufacturer" "Murata Power Solutions" (at 347.98 35.56 0) (hide yes) (effects (font (size 1.27 1.27)))) (property "LCSC" "C6823957" (at 347.98 35.56 0) (hide yes) (effects (font (size 1.27 1.27)))) (property "Assembly" "JLC_SMT_TOP_SUPPLY_BLOCKED" (at 347.98 35.56 0) (hide yes) (effects (font (size 1.27 1.27))))
     (instances
       (project "buck"
@@
       )
     )
-    (property "Migration_Status" "PENDING / ORIGINAL RETAINED"
+    (property "Migration_Status" "REV B - PART FIXED BY RELEASE PLAN"
       (at 347.98 35.56 0)
       (effects
@@
       )
     )
-    (property "Electrical_Approval" "PENDING - NOT APPROVED"
+    (property "Electrical_Approval" "PENDING - PROTOTYPE BRING-UP; NOT ELECTRICALLY VALIDATED"
       (at 347.98 35.56 0)
       (effects
@@
       )
     )
-    (property "Footprint" "Buck_SMD:PCAP_SVP_E7_PAN"
+    (property "Footprint" "Buck_RevB:CP_Panasonic_SVPF_E7_Land"
       (at 347.98 78.74 0)
       (hide yes)
@@
       )
     )
-    (property "Migration_Status" "FOOTPRINT_ONLY / PROVISIONAL - REVIEW REQUIRED"
+    (property "Migration_Status" "REV B - LAND CORRECTED TO MANUFACTURER DRAWING"
       (at 347.98 78.74 0)
       (effects
@@
       )
     )
-    (property "Footprint" "Buck_SMD:PCAP_SVP_E7_PAN"
+    (property "Footprint" "Buck_RevB:CP_Panasonic_SVPF_E7_Land"
       (at 50.8 121.92 0)
       (hide yes)
@@
       )
     )
-    (property "Migration_Status" "FOOTPRINT_ONLY / PROVISIONAL - REVIEW REQUIRED"
+    (property "Migration_Status" "REV B - LAND CORRECTED TO MANUFACTURER DRAWING"
       (at 50.8 121.92 0)
       (effects
@@
       )
     )
-    (property "Value" "LOAD + / -"
+    (property "Value" "LOAD TB002-500-02BE"
       (at 248.92 85.28 0)
       (show_name no)
@@
       )
     )
-    (property "Footprint" "TerminalBlock_Phoenix:TerminalBlock_Phoenix_MKDS-1,5-2_1x02_P5.00mm_Horizontal"
+    (property "Footprint" "Buck_RevB:TerminalBlock_SameSky_TB002-500-02_1x02_P5.00mm"
       (at 248.92 78.74 0)
       (hide yes)
@@
       )
     )
-    (property "Datasheet" ""
+    (property "Datasheet" "https://www.sameskydevices.com/product/resource/tb002-500.pdf"
       (at 248.92 78.74 0)
       (show_name no)
@@
     (pin "2"
     )
+    (property "MPN" "TB002-500-02BE" (at 248.92 78.74 0) (hide yes) (effects (font (size 1.27 1.27)))) (property "Manufacturer" "Same Sky" (at 248.92 78.74 0) (hide yes) (effects (font (size 1.27 1.27)))) (property "LCSC" "C2757858" (at 248.92 78.74 0) (hide yes) (effects (font (size 1.27 1.27)))) (property "Assembly" "MANUAL_THT" (at 248.92 78.74 0) (hide yes) (effects (font (size 1.27 1.27))))
     (instances
       (project "buck"
@@
       )
     )
-    (property "Migration_Status" "PENDING / ORIGINAL RETAINED"
+    (property "Migration_Status" "REV B - PART FIXED BY RELEASE PLAN"
       (at 248.92 78.74 0)
       (effects
@@
       )
     )
-    (property "Electrical_Approval" "PENDING - NOT APPROVED"
+    (property "Electrical_Approval" "PENDING - PROTOTYPE BRING-UP; NOT ELECTRICALLY VALIDATED"
       (at 248.92 78.74 0)
       (effects
@@
       )
     )
-    (property "Value" "330uH >=3A Isat VERIFY"
+    (property "Value" "330uH 60B334C"
       (at 50.8 85.28 0)
       (show_name no)
@@
       )
     )
-    (property "Footprint" "Buck:Inductor_25mm_P10mm_VERIFY"
+    (property "Footprint" "Buck_RevB:L_Murata_6000B_27.0x23.5mm"
       (at 50.8 78.74 0)
       (hide yes)
@@
       )
     )
-    (property "Datasheet" ""
+    (property "Datasheet" "https://www.murata.com/products/power/power-magnetics (KMP_6000B_B01)"
       (at 50.8 78.74 0)
       (show_name no)
@@
     (pin "1"
     )
+    (property "MPN" "60B334C" (at 50.8 78.74 0) (hide yes) (effects (font (size 1.27 1.27)))) (property "Manufacturer" "Murata Power Solutions" (at 50.8 78.74 0) (hide yes) (effects (font (size 1.27 1.27)))) (property "LCSC" "C6823957" (at 50.8 78.74 0) (hide yes) (effects (font (size 1.27 1.27)))) (property "Assembly" "JLC_SMT_TOP_SUPPLY_BLOCKED" (at 50.8 78.74 0) (hide yes) (effects (font (size 1.27 1.27))))
     (instances
       (project "buck"
@@
       )
     )
-    (property "Migration_Status" "PENDING / ORIGINAL RETAINED"
+    (property "Migration_Status" "REV B - PART FIXED BY RELEASE PLAN"
       (at 50.8 78.74 0)
       (effects
@@
       )
     )
-    (property "Electrical_Approval" "PENDING - NOT APPROVED"
+    (property "Electrical_Approval" "PENDING - PROTOTYPE BRING-UP; NOT ELECTRICALLY VALIDATED"
       (at 50.8 78.74 0)
       (effects
@@
       )
     )
-    (property "Value" "10uF 35V low ESR"
+    (property "Value" "10uF 50V 50SVF10M"
       (at 347.98 128.46 0)
       (show_name no)
@@
       )
     )
-    (property "Footprint" "Buck_SMD:CAP_SVF_C6_PAN"
+    (property "Footprint" "Buck_RevB:CP_Panasonic_SVF_C6_Land"
       (at 347.98 121.92 0)
       (hide yes)
@@
       )
     )
-    (property "Migration_Status" "FOOTPRINT_ONLY / PROVISIONAL - REVIEW REQUIRED"
+    (property "Migration_Status" "REV B - LAND CORRECTED TO MANUFACTURER DRAWING"
       (at 347.98 121.92 0)
       (effects
@@
       )
     )
-    (property "Value" "IRFZ44N TO-220"
+    (property "Value" "IRFZ44NPBF"
       (at 149.86 42.1 0)
       (show_name no)
@@
       )
     )
-    (property "Footprint" "Package_TO_SOT_THT:TO-220-3_Vertical"
+    (property "Footprint" "Buck_RevB:TO-220-3_Vertical_Drill1.4"
       (at 149.86 35.56 0)
       (hide yes)
@@
       )
     )
-    (property "Datasheet" ""
+    (property "Datasheet" "https://www.infineon.com/assets/row/public/documents/24/49/infineon-irfz44n-datasheet-en.pdf"
       (at 149.86 35.56 0)
       (show_name no)
@@
     (pin "1"
     )
+    (property "MPN" "IRFZ44NPBF" (at 149.86 35.56 0) (hide yes) (effects (font (size 1.27 1.27)))) (property "Manufacturer" "Infineon" (at 149.86 35.56 0) (hide yes) (effects (font (size 1.27 1.27)))) (property "LCSC" "C2586" (at 149.86 35.56 0) (hide yes) (effects (font (size 1.27 1.27)))) (property "Assembly" "MANUAL_THT" (at 149.86 35.56 0) (hide yes) (effects (font (size 1.27 1.27))))
     (instances
       (project "buck"
@@
       )
     )
-    (property "Migration_Status" "PENDING / ORIGINAL RETAINED"
+    (property "Migration_Status" "REV B - PART FIXED BY RELEASE PLAN"
       (at 149.86 35.56 0)
       (effects
@@
       )
     )
-    (property "Electrical_Approval" "PENDING - NOT APPROVED"
+    (property "Electrical_Approval" "PENDING - PROTOTYPE BRING-UP; NOT ELECTRICALLY VALIDATED"
       (at 149.86 35.56 0)
       (effects

Commit message: fix: make Buck Rev B orderable as a lab prototype
Order decisions after an external second opinion:
- Move the L1-L2-RS1-output chain 2 mm right: Q1 tab (VIN) to L1 SW clip
  clearance 1.28 -> 3.29 mm at maximum package dimensions; board rerouted,
  DRC 0 errors / 0 unconnected / 0 parity.
- L1/L2 (60B334C, no JLC/LCSC stock) leave the JLC BOM/CPL and are
  hand-soldered: 31 BOM lines, 62 placements, all with JLC stock.
- R10 -> UNI-ROYAL 0603WAF3092T5E (C23022), same 30.9k 1% 0603.
- Accept LM4040AIM3X-2.5/NOPB (same device per TI SNOS633N s.11).
- Document lab-only use: regulated 12 V, resistive load, supervised tests.

Co-Authored-By: Claude Opus 5.5 <noreply@anthropic.com>
Parts:
- L1, L2: Assembly JLC_SMT_TOP_SUPPLY_BLOCKED -> MANUAL_SMD_DNP_AT_JLC; Supply_Note (none) -> JLC/LCSC stock 0 on 2026-10-27; buy 60B334C (DigiKey 811-24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
Changed lines of the file:
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@@
     (pin "2"
     )
-    (property "MPN" "60B334C" (at 347.98 35.56 0) (hide yes) (effects (font (size 1.27 1.27)))) (property "Manufacturer" "Murata Power Solutions" (at 347.98 35.56 0) (hide yes) (effects (font (size 1.27 1.27)))) (property "LCSC" "C6823957" (at 347.98 35.56 0) (hide yes) (effects (font (size 1.27 1.27)))) (property "Assembly" "JLC_SMT_TOP_SUPPLY_BLOCKED" (at 347.98 35.56 0) (hide yes) (effects (font (size 1.27 1.27))))
+    (property "MPN" "60B334C" (at 347.98 35.56 0) (hide yes) (effects (font (size 1.27 1.27)))) (property "Manufacturer" "Murata Power Solutions" (at 347.98 35.56 0) (hide yes) (effects (font (size 1.27 1.27)))) (property "LCSC" "C6823957" (at 347.98 35.56 0) (hide yes) (effects (font (size 1.27 1.27)))) (property "Assembly" "MANUAL_SMD_DNP_AT_JLC" (at 347.98 35.56 0) (hide yes) (effects (font (size 1.27 1.27))))
+    (property "Supply_Note" "JLC/LCSC stock 0 on 2026-10-27; buy 60B334C (DigiKey 811-2464-ND) and hand-solder" (at 347.98 35.56 0) (hide yes) (effects (font (size 1.27 1.27))))
     (instances
       (project "buck"
@@
     (pin "1"
     )
-    (property "MPN" "60B334C" (at 50.8 78.74 0) (hide yes) (effects (font (size 1.27 1.27)))) (property "Manufacturer" "Murata Power Solutions" (at 50.8 78.74 0) (hide yes) (effects (font (size 1.27 1.27)))) (property "LCSC" "C6823957" (at 50.8 78.74 0) (hide yes) (effects (font (size 1.27 1.27)))) (property "Assembly" "JLC_SMT_TOP_SUPPLY_BLOCKED" (at 50.8 78.74 0) (hide yes) (effects (font (size 1.27 1.27))))
+    (property "MPN" "60B334C" (at 50.8 78.74 0) (hide yes) (effects (font (size 1.27 1.27)))) (property "Manufacturer" "Murata Power Solutions" (at 50.8 78.74 0) (hide yes) (effects (font (size 1.27 1.27)))) (property "LCSC" "C6823957" (at 50.8 78.74 0) (hide yes) (effects (font (size 1.27 1.27)))) (property "Assembly" "MANUAL_SMD_DNP_AT_JLC" (at 50.8 78.74 0) (hide yes) (effects (font (size 1.27 1.27))))
+    (property "Supply_Note" "JLC/LCSC stock 0 on 2026-10-27; buy 60B334C (DigiKey 811-2464-ND) and hand-solder" (at 50.8 78.74 0) (hide yes) (effects (font (size 1.27 1.27))))
     (instances
       (project "buck"
