File: project/pcb/redesign/buck_1.kicad_sch (KiCad schematic)
At the start: 12 parts, among them J1 12V IN TB002-500-02BE, J2 LOAD TB002-500-02BE, Q1 IRFZ44NPBF

Commit message: feat: replace Buck Rev B L1+L2 with a single JLC-placed 60B684C
L1+L2 (2 x Murata 60B334C in series) have no JLCPCB/LCSC stock, which
forced buying them at DigiKey and hand-soldering. A single Murata
60B684C (680 uH, 3 A, 135 mOhm, C6095796, JLC stock 17) from the same
6000B series uses the same drawing and land, so JLCPCB can place it.

- Schematic: L1 becomes 60B684C, L2 and the LMID net are removed and
  L1.2 joins IP (revb_tools/sch_single_inductor.py). ERC 0 errors;
  netdiff shows only those three changes.
- PCB: L2 removed, 3.5 mm F.Cu track from L1 pad 2 to the outer end of
  RS1; Kelvin traces and the 3.285 mm Q1 tab to L1 gap are unchanged.
  DRC 0 errors / 0 unconnected / 0 parity, same 3 justified width
  warnings. Stale LMID references removed from the SW width rule and
  netclass patterns.
- Package: BOM 32 lines / CPL 63 placements, all lines in JLC stock,
  manual list now only J1, J2, J3, Q1, D2. Hashes regenerated.
- Docs: +3 % inductance vs the 660 uH assignment value, losses, ripple,
  first power-on L1 check (578-782 uH, <= 135 mOhm) and the portal
  check that JLC accepts the 37 g / 20 mm part.

BUCK_BOARD_REVIEWED stays 0; firmware unchanged.

Co-Authored-By: Claude Opus 5.5 <noreply@anthropic.com>
Parts:
- removed L2: 330uH 60B334C, Buck_RevB:L_Murata_6000B_27.0x23.5mm, symbol Buck:L2
- L1: value 330uH 60B334C -> 680uH 60B684C; Assembly MANUAL_SMD_DNP_AT_JLC -> JLC_SMT_TOP; Commercial_URL (none) -> https://jlcpcb.com/partdetail/C6095796; LCSC C6823957 -> C6095796; MPN 60B334C -> 60B684C; Migration_Status REV B - PART FIXED BY RELEASE PLAN -> REV B - SINGLE 680uH INDUCTOR; Supply_Note JLC/LCSC stock 0 on 2026-10-27; buy 60B334C (DigiKey 811-24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 -> Replaces 2 x 60B334C (no JLC/LCSC stock); JLC stock 17 on 2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
Connections:
- net LMID is gone; now on net IP: L1.2
Changed lines of the file:
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@@
-  (wire
-    (pts
-      (xy 63.5 78.74)
-      (xy 68.58 78.74)
-    )
-    (stroke
-      (width 0)
-      (type default)
-    )
-  )
   (wire
     (pts
@@
   (wire
     (pts
-      (xy 38.1 78.74)
-      (xy 33.02 78.74)
-    )
-    (stroke
-      (width 0)
-      (type default)
-    )
-  )
-  (wire
-    (pts
       (xy 38.1 121.92)
       (xy 33.02 121.92)
@@
     )
   )
-  (global_label "LMID"
+  (global_label "IP"
     (shape passive)
     (at 365.76 35.56 0)
@@
     )
   )
-  (global_label "IP"
-    (shape passive)
-    (at 68.58 78.74 0)
+  (global_label "GND"
+    (shape passive)
+    (at 68.58 121.92 0)
     (effects
       (font
@@
     )
     (property "Intersheetrefs" "${INTERSHEET_REFS}"
-      (at 68.58 78.74 0)
+      (at 68.58 121.92 0)
       (hide yes)
       (show_name no)
@@
   (global_label "GND"
     (shape passive)
-    (at 68.58 121.92 0)
+    (at 68.58 35.56 0)
     (effects
       (font
@@
     )
     (property "Intersheetrefs" "${INTERSHEET_REFS}"
-      (at 68.58 121.92 0)
+      (at 68.58 35.56 0)
       (hide yes)
       (show_name no)
@@
   (global_label "GND"
     (shape passive)
-    (at 68.58 35.56 0)
+    (at 365.76 78.74 0)
     (effects
       (font
@@
     )
     (property "Intersheetrefs" "${INTERSHEET_REFS}"
-      (at 68.58 35.56 0)
-      (hide yes)
-      (show_name no)
-      (do_not_autoplace no)
-      (effects
-        (font
-          (size 1.27 1.27)
-        )
-      )
-    )
-  )
-  (global_label "GND"
-    (shape passive)
-    (at 365.76 78.74 0)
-    (effects
-      (font
-        (size 0.85 0.85)
-      )
-      (justify left)
-    )
-    (property "Intersheetrefs" "${INTERSHEET_REFS}"
       (at 365.76 78.74 0)
       (hide yes)
@@
     (property "Intersheetrefs" "${INTERSHEET_REFS}"
       (at 132.08 35.56 0)
-      (hide yes)
-      (show_name no)
-      (do_not_autoplace no)
-      (effects
-        (font
-          (size 1.27 1.27)
-        )
-      )
-    )
-  )
-  (global_label "LMID"
-    (shape passive)
-    (at 33.02 78.74 180)
-    (effects
-      (font
-        (size 0.85 0.85)
-      )
-      (justify right)
-    )
-    (property "Intersheetrefs" "${INTERSHEET_REFS}"
-      (at 33.02 78.74 0)
       (hide yes)
       (show_name no)
@@
       )
     )
-    (property "Value" "330uH 60B334C"
+    (property "Value" "680uH 60B684C"
       (at 347.98 42.1 0)
       (show_name no)
@@
     (pin "2"
     )
-    (property "MPN" "60B334C" (at 347.98 35.56 0) (hide yes) (effects (font (size 1.27 1.27)))) (property "Manufacturer" "Murata Power Solutions" (at 347.98 35.56 0) (hide yes) (effects (font (size 1.27 1.27)))) (property "LCSC" "C6823957" (at 347.98 35.56 0) (hide yes) (effects (font (size 1.27 1.27)))) (property "Assembly" "MANUAL_SMD_DNP_AT_JLC" (at 347.98 35.56 0) (hide yes) (effects (font (size 1.27 1.27))))
-    (property "Supply_Note" "JLC/LCSC stock 0 on 2026-10-27; buy 60B334C (DigiKey 811-2464-ND) and hand-solder" (at 347.98 35.56 0) (hide yes) (effects (font (size 1.27 1.27))))
+    (property "MPN" "60B684C" (at 347.98 35.56 0) (hide yes) (effects (font (size 1.27 1.27)))) (property "Manufacturer" "Murata Power Solutions" (at 347.98 35.56 0) (hide yes) (effects (font (size 1.27 1.27)))) (property "LCSC" "C6095796" (at 347.98 35.56 0) (hide yes) (effects (font (size 1.27 1.27)))) (property "Assembly" "JLC_SMT_TOP" (at 347.98 35.56 0) (hide yes) (effects (font (size 1.27 1.27))))
+    (property "Supply_Note" "Replaces 2 x 60B334C (no JLC/LCSC stock); JLC stock 17 on 2026-10-27; 680 uH = +3 % vs 660 uH" (at 347.98 35.56 0) (hide yes) (effects (font (size 1.27 1.27))))
+    (property "Commercial_URL" "https://jlcpcb.com/partdetail/C6095796" (at 347.98 35.56 0) (hide yes) (effects (font (size 1.27 1.27))))
     (instances
       (project "buck"
@@
       )
     )
-    (property "Migration_Status" "REV B - PART FIXED BY RELEASE PLAN"
+    (property "Migration_Status" "REV B - SINGLE 680uH INDUCTOR"
       (at 347.98 35.56 0)
       (effects
@@
       (effects
         (font
-          (size 1 1)
-        )
-        (hide yes)
-      )
-    )
-  )
-  (symbol
-    (lib_id "Buck:L2")
-    (at 50.8 78.74 0)
-    (unit 1)
-    (body_style 1)
-    (exclude_from_sim no)
-    (in_bom yes)
-    (on_board yes)
-    (in_pos_files yes)
-    (dnp no)
-    (property "Reference" "L2"
-      (at 50.8 72.2 0)
-      (show_name no)
-      (do_not_autoplace no)
-      (effects
-        (font
-          (size 1.27 1.27)
-        )
-      )
-    )
-    (property "Value" "330uH 60B334C"
-      (at 50.8 85.28 0)
-      (show_name no)
-      (do_not_autoplace no)
-      (effects
-        (font
-          (size 0.95 0.95)
-        )
-      )
-    )
-    (property "Footprint" "Buck_RevB:L_Murata_6000B_27.0x23.5mm"
-      (at 50.8 78.74 0)
-      (hide yes)
-      (show_name no)
-      (do_not_autoplace no)
-      (effects
-        (font
-          (size 1 1)
-        )
-      )
-    )
-    (property "Datasheet" "https://www.murata.com/products/power/power-magnetics (KMP_6000B_B01)"
-      (at 50.8 78.74 0)
-      (show_name no)
-      (do_not_autoplace no)
-      (effects
-        (font
-          (size 1.27 1.27)
-        )
-      )
-    )
-    (property "Description" ""
-      (at 50.8 78.74 0)
-      (show_name no)
-      (do_not_autoplace no)
-      (effects
-        (font
-          (size 1.27 1.27)
-        )
-      )
-    )
-    (pin "2"
-    )
-    (pin "1"
-    )
-    (property "MPN" "60B334C" (at 50.8 78.74 0) (hide yes) (effects (font (size 1.27 1.27)))) (property "Manufacturer" "Murata Power Solutions" (at 50.8 78.74 0) (hide yes) (effects (font (size 1.27 1.27)))) (property "LCSC" "C6823957" (at 50.8 78.74 0) (hide yes) (effects (font (size 1.27 1.27)))) (property "Assembly" "MANUAL_SMD_DNP_AT_JLC" (at 50.8 78.74 0) (hide yes) (effects (font (size 1.27 1.27))))
-    (property "Supply_Note" "JLC/LCSC stock 0 on 2026-10-27; buy 60B334C (DigiKey 811-2464-ND) and hand-solder" (at 50.8 78.74 0) (hide yes) (effects (font (size 1.27 1.27))))
-    (instances
-      (project "buck"
-        (path "/94b2b377-c0d1-5fce-91fa-ae8f86f36484/e29e3f6c-31ac-5304-9825-4ea039ba59c0"
-          (reference "L2")
-          (unit 1)
-        )
-      )
-    )
-    (property "Migration_Status" "REV B - PART FIXED BY RELEASE PLAN"
-      (at 50.8 78.74 0)
-      (effects
-        (font
-          (size 1 1)
-        )
-        (hide yes)
-      )
-    )
-    (property "Candidate_MPN" "Murata 60B334C"
-      (at 50.8 78.74 0)
-      (effects
-        (font
-          (size 1 1)
-        )
-        (hide yes)
-      )
-    )
-    (property "Candidate_LCSC" "C6823957"
-      (at 50.8 78.74 0)
-      (effects
-        (font
-          (size 1 1)
-        )
-        (hide yes)
-      )
-    )
-    (property "Electrical_Approval" "PENDING - PROTOTYPE BRING-UP; NOT ELECTRICALLY VALIDATED"
-      (at 50.8 78.74 0)
-      (effects
-        (font
-          (size 1 1)
-        )
-        (hide yes)
-      )
-    )
-    (property "Migration_Notes" "Igual L1; se conserva huella THT histórica solo como original NO MIGRADO. Comprobar influencia de proximidad/acoplamiento: L_eq = L1+L2±2M. Validar I de saturación por condición de 80 % del nominal y temperatura."
-      (at 50.8 78.74 0)
-      (effects
-        (font

Commit message: fix: hand-solder Buck Rev B L1 instead of JLC placement
A second, informal external review of 6908b4d flagged two problems with
JLCPCB placing the single 60B684C. Both were verified:

- Murata KMP_6000B_B01 p.1 limits peak reflow to 245 C (J-STD-020D.1),
  while JLCPCB Economic PCBA reflows at 255 +/- 5 C, not adjustable
  (Standard PCBA: 240 +/- 5 C).
- The L1 body ends 0.48 mm from the bottom board edge (pcbnew F.Fab);
  no other SMD part is closer than 4.17 mm.

L1 becomes MANUAL_SMD_DNP_AT_JLC (revb_tools/sch_l1_hand_solder.py;
symbol and footprint fields synced so schematic parity stays at 0).
Order Economic PCBA for the other 62 SMD parts and buy the 60B684C
separately (LCSC C6095796). Copper, mask and paste are unchanged, so the
Gerbers match 6908b4d apart from headers and the L1 pads arrive tinned.

ERC 0 errors / 2 UART warnings; DRC 0 errors, 0 unconnected, 0 parity,
same 3 justified width warnings; BOM 31 lines / CPL 62, all in stock.
The overcurrent trip (~2.0 A peak) stays below the 3 A rating. Docs add
the hand-soldering steps, the Standard PCBA alternative and the edge
handling note. BUCK_BOARD_REVIEWED stays 0.

Co-Authored-By: Claude Opus 5.5 <noreply@anthropic.com>
Parts:
- L1: Assembly JLC_SMT_TOP -> MANUAL_SMD_DNP_AT_JLC; Migration_Status REV B - SINGLE 680uH INDUCTOR -> REV B - SINGLE 680uH INDUCTOR, HAND-SOLDERED; Supply_Note Replaces 2 x 60B334C (no JLC/LCSC stock); JLC stock 17 on 2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 -> Not placed by JLC: 6000B peak reflow 245 C < Economic PCBA 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
Changed lines of the file:
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@@
     (pin "2"
     )
-    (property "MPN" "60B684C" (at 347.98 35.56 0) (hide yes) (effects (font (size 1.27 1.27)))) (property "Manufacturer" "Murata Power Solutions" (at 347.98 35.56 0) (hide yes) (effects (font (size 1.27 1.27)))) (property "LCSC" "C6095796" (at 347.98 35.56 0) (hide yes) (effects (font (size 1.27 1.27)))) (property "Assembly" "JLC_SMT_TOP" (at 347.98 35.56 0) (hide yes) (effects (font (size 1.27 1.27))))
-    (property "Supply_Note" "Replaces 2 x 60B334C (no JLC/LCSC stock); JLC stock 17 on 2026-10-27; 680 uH = +3 % vs 660 uH" (at 347.98 35.56 0) (hide yes) (effects (font (size 1.27 1.27))))
+    (property "MPN" "60B684C" (at 347.98 35.56 0) (hide yes) (effects (font (size 1.27 1.27)))) (property "Manufacturer" "Murata Power Solutions" (at 347.98 35.56 0) (hide yes) (effects (font (size 1.27 1.27)))) (property "LCSC" "C6095796" (at 347.98 35.56 0) (hide yes) (effects (font (size 1.27 1.27)))) (property "Assembly" "MANUAL_SMD_DNP_AT_JLC" (at 347.98 35.56 0) (hide yes) (effects (font (size 1.27 1.27))))
+    (property "Supply_Note" "Not placed by JLC: 6000B peak reflow 245 C < Economic PCBA 255+/-5 C and body 0.48 mm from board edge; buy 60B684C (LCSC C6095796, stock 17 on 2026-10-27) and hand-solder" (at 347.98 35.56 0) (hide yes) (effects (font (size 1.27 1.27))))
     (property "Commercial_URL" "https://jlcpcb.com/partdetail/C6095796" (at 347.98 35.56 0) (hide yes) (effects (font (size 1.27 1.27))))
     (instances
@@
       )
     )
-    (property "Migration_Status" "REV B - SINGLE 680uH INDUCTOR"
+    (property "Migration_Status" "REV B - SINGLE 680uH INDUCTOR, HAND-SOLDERED"
       (at 347.98 35.56 0)
       (effects
